File: pcb/common-ibc.kicad_pcb (KiCad board)
At the start: 4 copper layers, 67 x 65 mm, 103 parts, among them J1 XILINX_JTAG, J10 U.FL, J11 MOLEX_0039291087, J2 MOLEX_0039291067, J3 GROUND, J4 GROUND, J5 MOLEX_0532610571, J6 U.FL, J7 U.FL, J8 U.FL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

Commit message: Final version sent to fab for quotes
Routing:
- net /3V3_SB: track 193.2 -> 194.3 mm
Changed lines of the file:
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@@
 		(allow_soldermask_bridges_in_footprints no)
 		(pcbplotparams
-			(layerselection 0x00010fc_ffffffff)
+			(layerselection 0x00210fc_ffffffff)
 			(plot_on_all_layers_selection 0x0000000_00000000)
 			(disableapertmacros no)
@@
 			(usegerberattributes yes)
 			(usegerberadvancedattributes yes)
-			(creategerberjobfile yes)
+			(creategerberjobfile no)
 			(dashed_line_dash_ratio 12.000000)
 			(dashed_line_gap_ratio 3.000000)
@@
 			(outputformat 1)
 			(mirror no)
-			(drillshape 1)
+			(drillshape 0)
 			(scaleselection 1)
-			(outputdirectory "")
+			(outputdirectory "output/")
 		)
 	)
@@
 		(at 41.25 45.7 -90)
 		(property "Reference" "U8"
-			(at 0.2 1.65 270)
+			(at 0.2 1.65 -90)
 			(unlocked yes)
 			(layer "F.SilkS")
@@
 		(at 95.6 48 -90)
 		(property "Reference" "J5"
-			(at 0 2.000001 270)
+			(at 0 2.000001 -90)
 			(unlocked yes)
 			(layer "F.SilkS")
@@
 		)
 		(property "Value" "MI0603J601R-10"
-			(at 0 -1.75 360)
+			(at 0 -1.75 0)
 			(unlocked yes)
 			(layer "B.SilkS")
@@
 	)
 	(segment
-		(start 89.3 48.725)
-		(end 93.341636 48.725)
+		(start 63.6 77.2)
+		(end 63.6 77.95)
 		(width 0.125)
 		(layer "In2.Cu")
@@
 	)
 	(segment
-		(start 45 58.6)
-		(end 48.6 62.2)
+		(start 63.9 76.9)
+		(end 63.6 77.2)
 		(width 0.125)
 		(layer "In2.Cu")
@@
 	)
 	(segment
-		(start 93.341636 48.725)
-		(end 94.5 49.883364)
+		(start 49 62.2)
+		(end 49.008318 62.208318)
 		(width 0.125)
 		(layer "In2.Cu")
@@
 	)
 	(segment
+		(start 49.008318 62.208318)
+		(end 55.508318 62.208318)
+		(width 0.125)
+		(layer "In2.Cu")
+		(net 3)
+	)
+	(segment
 		(start 83.5 44.85)
 		(end 83.5 46.5)
@@
 	)
 	(segment
-		(start 49.008318 62.208318)
-		(end 54.791682 62.208318)
+		(start 45 58.6)
+		(end 48.6 62.2)
 		(width 0.125)
 		(layer "In2.Cu")
@@
 	)
 	(segment
-		(start 64.75 77)
-		(end 64.75 81)
+		(start 71 82)
+		(end 70.583364 81.583364)
 		(width 0.125)
 		(layer "In2.Cu")
@@
 	)
 	(segment
-		(start 71 82)
-		(end 70.583364 81.583364)
+		(start 64.25 75.55)
+		(end 63.9 75.9)
 		(width 0.125)
 		(layer "In2.Cu")
@@
 	)
 	(segment
+		(start 92.725 48.725)
+		(end 94.5 50.5)
+		(width 0.125)
+		(layer "In2.Cu")
+		(net 3)
+	)
+	(segment
+		(start 55.508318 62.208318)
+		(end 58 64.7)
+		(width 0.125)
+		(layer "In2.Cu")
+		(net 3)
+	)
+	(segment
+		(start 64.75 79.1)
+		(end 64.75 79.4)
+		(width 0.125)
+		(layer "In2.Cu")
+		(net 3)
+	)
+	(segment
 		(start 89.25 51.35)
 		(end 89.25 53.5)
@@
 	)
 	(segment
-		(start 64.25 75.25)
-		(end 64.25 76.5)
+		(start 59.4 68.8)
+		(end 59.4 69.233364)
 		(width 0.125)
 		(layer "In2.Cu")
@@
 	)
 	(segment
-		(start 59.4 68.8)
-		(end 59.4 69.233364)
+		(start 63 82)
+		(end 63 81.3)
+		(width 0.125)
+		(layer "In2.Cu")
+		(net 3)
+	)
+	(segment
+		(start 64.75 79.55)
+		(end 64.75 79.4)
 		(width 0.125)
 		(layer "In2.Cu")
@@
 	)
 	(segment
-		(start 57.283364 64.7)
-		(end 59.1 64.7)
+		(start 64.25 75.25)
+		(end 64.25 75.55)
 		(width 0.125)
 		(layer "In2.Cu")
@@
 	)
 	(segment
-		(start 45 50.5)
-		(end 45 58.6)
-		(width 0.125)
-		(layer "In2.Cu")
-		(net 3)
-	)
-	(segment
 		(start 59.3875 68.7875)
 		(end 59.3875 64.9875)
@@
 	)
 	(segment
-		(start 65.4 81.583364)
-		(end 64.5 81.583364)
+		(start 63.6 77.95)
+		(end 64.75 79.1)
 		(width 0.125)
 		(layer "In2.Cu")
@@
 	)
 	(segment
-		(start 64.5 81.25)
-		(end 64.5 81.583364)
+		(start 89.3 48.725)
+		(end 92.725 48.725)
 		(width 0.125)
 		(layer "In2.Cu")
@@
 	)
 	(segment
-		(start 95.5 42.25)
-		(end 95.5 49.5)
+		(start 64.75 80.933364)
+		(end 65.4 81.583364)
 		(width 0.125)
 		(layer "In2.Cu")
@@
 	)
 	(segment
-		(start 83.5 44.516636)
-		(end 86.766636 41.25)
+		(start 95.5 42.25)
+		(end 95.5 49.5)
 		(width 0.125)
 		(layer "In2.Cu")
@@
 	)
 	(segment
-		(start 64.25 76.5)
-		(end 64.75 77)
+		(start 45 50.5)
+		(end 45 58.6)
 		(width 0.125)
 		(layer "In2.Cu")
@@
 	)
 	(segment
-		(start 83.25 50.75)
-		(end 81.25 48.75)
+		(start 83.5 44.516636)
+		(end 86.766636 41.25)
 		(width 0.125)
 		(layer "In2.Cu")
@@
 	)
 	(segment
-		(start 54.791682 62.208318)
-		(end 57.283364 64.7)
+		(start 83.25 50.75)
+		(end 81.25 48.75)
 		(width 0.125)
 		(layer "In2.Cu")
@@
 	)
 	(segment
-		(start 45.166636 50.5)
-		(end 45 50.5)
+		(start 63 81.3)
+		(end 64.75 79.55)
 		(width 0.125)
 		(layer "In2.Cu")
@@
 	)
 	(segment
-		(start 64.75 81)
-		(end 64.5 81.25)
+		(start 45.166636 50.5)
+		(end 45 50.5)
 		(width 0.125)
 		(layer "In2.Cu")
@@
 	)
 	(segment
-		(start 48.6 62.2)
-		(end 49 62.2)
+		(start 63.9 75.9)
+		(end 63.9 76.9)
 		(width 0.125)
 		(layer "In2.Cu")
@@
 	)
 	(segment
-		(start 94.5 49.883364)
-		(end 94.5 50.5)
+		(start 48.6 62.2)
+		(end 49 62.2)
 		(width 0.125)
 		(layer "In2.Cu")
@@
 	)
 	(segment
-		(start 64.5 81.583364)
-		(end 64.083364 82)
+		(start 47.4375 81.4375)
+		(end 62.4375 81.4375)
 		(width 0.125)
 		(layer "In2.Cu")
@@
 	)
 	(segment
-		(start 47.4375 81.4375)
-		(end 62.4375 81.4375)
+		(start 64.25 74.083364)
+		(end 64.25 75.25)
 		(width 0.125)
 		(layer "In2.Cu")
@@
 	)
 	(segment
-		(start 64.083364 82)
-		(end 63 82)
+		(start 36.8 49.2)
+		(end 36.3 49.7)
 		(width 0.125)
 		(layer "In2.Cu")
@@
 	)
 	(segment
-		(start 64.25 74.083364)
-		(end 64.25 75.25)
+		(start 83.5 46.5)
+		(end 81.25 48.75)
 		(width 0.125)
 		(layer "In2.Cu")
@@
 	)
 	(segment
-		(start 36.8 49.2)
-		(end 36.3 49.7)
+		(start 58 64.7)
+		(end 59.1 64.7)
 		(width 0.125)
 		(layer "In2.Cu")
@@
 	)
 	(segment
-		(start 83.5 46.5)
-		(end 81.25 48.75)
+		(start 64.75 79.4)
+		(end 64.75 80.933364)
 		(width 0.125)
 		(layer "In2.Cu")
@@
 		(width 0.125)
 		(layer "In2.Cu")
-		(net 3)
-	)
-	(segment
-		(start 49 62.2)
-		(end 49.008318 62.208318)
-		(width 0.125)
-		(layer "In2.Cu")

Commit message: Hopefully-mostly-done v0.5 layout
Parts:
- removed FL1: ACM90V-701-2PL-TL00, azonenberg_pcb:CMC_TDK_ACM90V
- removed Q1: SI7942DP, azonenberg_pcb:SOIC_8_3.9MM
- added C24: GA343DR7GD472KW01L, azonenberg_pcb:EIA_1812_CAP_NOSILK, F.Cu at (73.0, 32.0)
- added C27: 875105945001, azonenberg_pcb:CAP_AL_6.3MM_SMT, F.Cu at (81.5, 33.0)
- added C28: 10 nF, azonenberg_pcb:EIA_0402_CAP_NOSILK, B.Cu at (69.0, 40.5)
- added D6: PTVS58VP1UP,115, azonenberg_pcb:SOD128, F.Cu at (76.8, 25.2)
- added D7: ES2J-LTP, azonenberg_pcb:SMA, F.Cu at (73.0, 25.5)
- added R35: DNP, azonenberg_pcb:EIA_0402_RES_NOSILK, B.Cu at (69.0, 41.5)
- added R36: DNP, azonenberg_pcb:EIA_0603_RES_NOSILK, F.Cu at (76.8, 35.2)
- added R37: DNP, azonenberg_pcb:EIA_0402_RES_NOSILK, F.Cu at (75.5, 35.0)
- added R38: 17.8K, azonenberg_pcb:EIA_0402_RES_NOSILK, B.Cu at (69.0, 39.0)
- added TP3: TESTPOINT, azonenberg_pcb:TESTPOINT_SMT_0.5MM, F.Cu at (73.8, 45.8)
- R27: value 576K -> DNP; footprint azonenberg_pcb:EIA_0402_RES_NOSILK -> azonenberg_pcb:EIA_0805_CAP_NOSILK
- R28: value 10M -> 806K; footprint azonenberg_pcb:EIA_0402_RES_NOSILK -> azonenberg_pcb:EIA_0603_RES_NOSILK
- R29: value 49.9K -> 620; moved to B.Cu
- R30: value 187K -> 6.49K; moved to B.Cu
- R33: value 10M -> 9.09K; moved to B.Cu
- R34: value 23.2K -> 20K
- U1: value LTC4367 -> TPS16630; footprint azonenberg_pcb:DFN_8_0.5MM_3x3MM -> azonenberg_pcb:QFN_24_0.5MM_4x4MM
- moved R1 23.2 mm to (87.2, 23.8), turned to -90 degrees
- moved R34 22.1 mm to (73.0, 44.5)
- moved R33 21.9 mm to (70.8, 41.0)
- moved R29 21.2 mm to (70.5, 38.5), turned to -90 degrees
- moved R28 18.7 mm to (73.8, 37.0)
- moved R30 17.5 mm to (72.0, 38.0)
- moved TP2 16.3 mm to (74.5, 44.0)
- moved U1 16.2 mm to (74.5, 40.8), turned to -90 degrees
- moved R27 15.3 mm to (78.5, 39.0), turned to -90 degrees
- moved FB1 12.4 mm to (80.5, 26.0), turned to -90 degrees
Connections:
- FB1 pad 2: /48V_PROT -> /48V_FUSED
- J2 pad 4: /GND_RAW -> /GND
- J2 pad 5: /GND_RAW -> /GND
- J2 pad 6: /GND_RAW -> /GND
- R1 pad 2: /48V0 -> /48V0_SHOUT
- R27 pad 1: /48V_CMC -> /48V0_SHOUT
- R27 pad 2: Net-(U1-~{SHDN}) -> /48V0
- R28 pad 1: Net-(U1-~{SHDN}) -> /48V0_SHOUT
- R28 pad 2: Net-(R28-Pad2) -> /VUVLO
- R29 pad 1: Net-(U1-UV) -> Net-(R29-Pad1)
- R29 pad 2: Net-(R29-Pad2) -> /VOVP
- R30 pad 1: Net-(U1-OV) -> /VUVLO
- R30 pad 2: /GND -> Net-(R29-Pad1)
- R33 pad 1: Net-(R28-Pad2) -> /ILIM
- R33 pad 2: Net-(U1-UV) -> /GND
- R34 pad 1: Net-(R29-Pad2) -> /48V0_IMON
- R34 pad 2: Net-(U1-OV) -> /GND
- TP2 pad 1: /PROT_FAULT -> /48V0_GOOD
- U1 pad 1: /48V_CMC -> /48V0_SHOUT
- U1 pad 2: Net-(U1-UV) -> /48V0_SHOUT
- U1 pad 3: Net-(U1-OV) -> (no net)
- U1 pad 4: /GND -> (no net)
- U1 pad 5: Net-(U1-~{SHDN}) -> /48V0_SHOUT
- U1 pad 6: /PROT_FAULT -> /VUVLO
- U1 pad 7: /48V_PROT -> /VOVP
- U1 pad 8: /PROT_GATE -> /GND
- U9 pad 15: unconnected-(U9A-PA5-Pad15) -> /48V0_IMON
- U9 pad 18: unconnected-(U9B-PB0-Pad18) -> /3V3_SB
Routing:
- net /GND_RAW: track 39.9 -> 0.00 mm
- net /48V0_IMON: track 0.00 -> 36.0 mm, vias 0 -> 2
- net /48V0_SHOUT: track 0.00 -> 32.3 mm
- net /48V_SHUNT_N: track 3.01 -> 33.7 mm
- net /48V_CMC: track 28.5 -> 0.00 mm
- net /GND: track 468.5 -> 489.1 mm, vias 221 -> 345
- net /48V_SHUNT_P: track 2.97 -> 23.4 mm
- net /48V_PROT: track 16.3 -> 0.00 mm, vias 2 -> 0
- net /PROT_GATE: track 14.4 -> 0.00 mm
- net /48V0: track 39.7 -> 53.1 mm
- net /TPS_SHDN: track 0.00 -> 13.4 mm, vias 0 -> 2
- net /48V_FUSED: track 8.03 -> 20.4 mm
- net /I2C_SCL: track 119.8 -> 107.9 mm, vias 5 -> 7
- net /I2C_SDA: track 128.0 -> 116.3 mm, vias 5 -> 7
- net Net-(U1-~{SHDN}): track 8.79 -> 0.00 mm, vias 2 -> 0
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- added copper zone on F.Cu, net /48V0_SHOUT
- added copper zone on In2.Cu, net /GND
- removed copper zone on F.Cu, net /48V0_MIDPROT
- removed copper zone on F.Cu, net /48V_CMC
- removed copper zone on F.Cu, net /48V_PROT
- removed copper zone on F.Cu, net /48V_SHIN
- removed copper zone on F.Cu, net /GND_RAW
Other:
- board text added: "48-12V IBC A. Zonenberg 2024-08-10 v0.5"
- board text removed: "48-12V IBC A. Zonenberg 2024-07-06 v0.4"
