File: pcb/common-ibc.kicad_pcb (KiCad board)
At the start: 4 copper layers, 67 x 65 mm, 111 parts, among them J1 XILINX_JTAG, J10 U.FL, J11 MOLEX_0039291087, J2 MOLEX_0039291067, J3 GROUND, J4 GROUND, J5 MOLEX_0532610571, J6 U.FL, J7 U.FL, J8 U.FL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

Commit message: Final v0.5 IBC design going to fab for quotes
Parts:
- added D4: PTVS58VP1UP,115, azonenberg_pcb:SOD128, F.Cu at (92.0, 28.2)
Routing:
- net /GND: track 489.1 -> 489.9 mm, vias 345 -> 367
- net /48V_RAW: track 31.9 -> 31.4 mm
- added copper zone on F.Cu, net /48V_RAW
- added copper zone on F.Cu, net /48V_SHIN
Other:
- board text added: "48-12V IBC A. Zonenberg 2024-08-12 v0.5"
- board text removed: "48-12V IBC A. Zonenberg 2024-08-10 v0.5"
